File: hw/bx-hub75/bx-hub75.sch (KiCad schematic (older format))
At the start: 17 parts, among them J1 DB9_Male, J2 Barrel_Jack_MountingPin, U1 74HCT541, U2 74HCT541, U3 LD1117S33TR_SOT223

Commit message: hw/bx-hub75: release V0.4.
Parts:
- removed 1:32: E Line Enable, Connector_PinHeader_2.54mm:PinHeader_1x03_P2.54mm_Vertical, symbol Jumper:Jumper_3_Bridged12
- removed J2: Barrel_Jack_MountingPin, Connector_BarrelJack:BarrelJack_CUI_PJ-063AH_Horizontal, symbol Connector:Barrel_Jack_MountingPin
- removed U1, U2: 74HCT541, Package_SO:SOIC-20W_7.5x12.8mm_P1.27mm, symbol 74xx:74HCT541
- added J2: Barrel_Jack, Connector_BarrelJack:BarrelJack_Wuerth_6941xx301002, symbol Connector:Barrel_Jack
- added R10, R11, R12, R13, R14, R15, R16, R3, R4, R5, R6, R7, R8, R9: 33, Resistor_SMD:R_0805_2012Metric_Pad1.15x1.40mm_HandSolder, symbol Device:R
- added U1, U2: 74LVC4245A, Package_SO:SOIC-24W_7.5x15.4mm_P1.27mm, symbol Random:74LVC4245A
- CHAIN1: footprint Random:HUB75_HEADER -> Connector_IDC:IDC-Header_2x08_P2.54mm_Vertical
Connections:
- net +3V3: now also U1.1 (VCCA), U1.2 (DIR), U2.1 (VCCA), U2.2 (DIR)
- net +5V: now also J2.1, U1.23 (VCCB), U1.24 (VCCB), U2.23 (VCCB), U2.24 (VCCB)
- net A: now also U1.7 (A4)
- net B: now also U2.5 (A2)
- net B1: now also U1.4 (A1)
- net B2: now also U1.6 (A3)
- net C: now also U1.8 (A5)
- net CLK: now also U1.9 (A6)
- net D: now also U2.4 (A1)
- net E: now also FPGA1.13 (IO_12), U2.6 (A3); no longer FPGA1.25 (IO_24)
- net G1: now also FPGA1.24 (IO_23), U2.8 (A5); no longer FPGA1.14 (IO_13)
- net G2: now also FPGA1.14 (IO_13), U2.7 (A4); no longer FPGA1.13 (IO_12)
- net GND: now also J2.2, U1.11 (GND), U1.12 (GND), U1.13 (GND), U1.22 (~OE), U2.10 (A7), U2.11 (GND), U2.12 (GND), U2.13 (GND), U2.22 (~OE), U2.9 (A6)
- net LAT: now also U2.3 (A0)
- net OE: now also U1.10 (A7)
- net R1: now also U1.3 (A0)
- net R2: now also U1.5 (A2)
- net RX: now also FPGA1.15 (IO_14); no longer FPGA1.16 (IO_15)
- net RX+: now also J1.1, R1.2; no longer J1.2, R1.1
- net RX-: now also J1.2, R1.1; no longer J1.1, R1.2
- net TX: now also FPGA1.16 (IO_15); no longer FPGA1.15 (IO_14)
- net TX+: now also RS485.5 (Y); no longer RS485.6 (Z)
- net TX-: now also RS485.6 (Z); no longer RS485.5 (Y)
- net at CHAIN1.1 (R1): now also R3.1
- net at CHAIN1.10 (B): now also R14.2
- net at CHAIN1.11 (C): now also R8.1
- net at CHAIN1.12 (D): now also R15.2
- net at CHAIN1.13 (CLK): now also R9.1
- net at CHAIN1.14 (LAT): now also R16.2
- net at CHAIN1.15 (OE): now also R10.1
- net at CHAIN1.2 (G1): now also R11.2
- net at CHAIN1.3 (B1): now also R4.1
- net at CHAIN1.5 (R2): now also R5.1
- net at CHAIN1.6 (G2): now also R12.2
- net at CHAIN1.7 (B2): now also R6.1
- net at CHAIN1.9 (A): now also R7.1
- net E_PIN: no longer names the net of CHAIN1.8 (E)
- net E_PIN: now also R13.2
- new net: R10.2, U1.14 (B7)
- new net: R9.2, U1.15 (B6)
- new net: R8.2, U1.16 (B5)
- new net: R7.2, U1.17 (B4)
- new net: R6.2, U1.18 (B3)
- new net: R5.2, U1.19 (B2)
- new net: R4.2, U1.20 (B1)
- new net: R3.2, U1.21 (B0)
- new net: R11.1, U2.16 (B5)
- new net: R12.1, U2.17 (B4)
- new net: R13.1, U2.18 (B3)
- new net: R14.1, U2.19 (B2)
- new net: R15.1, U2.20 (B1)
- new net: R16.1, U2.21 (B0)
