File: hw/rs485-breakout/rs485-breakout.sch (KiCad schematic (older format))
At the start: 18 parts, among them J1 DB9_Female, J2 DB9_Female, J3 DB9_Female, J4 DB9_Female, U1 SN65HVD77D, U2 SN65HVD77D, U3 SN65HVD77D, U4 SN65HVD77D

Commit message: hw/bx-hub75: release V0.4.
Parts:
- renumbered C2 to C1
Changed lines of the file:
@@
 $EndComp
 $Comp
-L Device:C C2
+L Device:C C1
 U 1 1 5C2DA94F
 P 2200 3950
-F 0 "C2" H 2315 3996 50  0000 L CNN
+F 0 "C1" H 2315 3996 50  0000 L CNN
 F 1 "100uf" H 2315 3905 50  0000 L CNN
 F 2 "Capacitor_SMD:CP_Elec_5x5.4" H 2238 3800 50  0001 C CNN
